Commit message: Publish rate of controllers updated to 5

File: src/racecar-simulator/racecar_description/urdf/racecar_2.xacro (robot description, xacro)
@@ -11,5 +11,5 @@
   </link>
   <joint name="base_link_joint" type="fixed">
-    <origin xyz="1 0 0.05" rpy="0 0 0" />
+    <origin xyz="0 0 0.05" rpy="0 0 0" />
     <parent link="base_link" />
     <child link="chassis" />
@@ -43,5 +43,5 @@
     <child link="left_rear_wheel" />
     <axis xyz="0 0 -1" />
-    <limit effort="10" velocity="100" />
+    <limit effort="10" velocity="1000" />
   </joint>
   <xacro:wheel_transmission name="left_rear_wheel" />
@@ -64,5 +64,5 @@
     <child link="right_rear_wheel" />
     <axis xyz="0 0 -1" />
-    <limit effort="10" velocity="100" />
+    <limit effort="10" velocity="1000" />
   </joint>
   <xacro:wheel_transmission name="right_rear_wheel" />
@@ -82,5 +82,5 @@
     <child link="left_steering_hinge" />
     <axis xyz="-1 0 0" />
-    <limit lower="-1.0" upper="1.0" effort="10" velocity="100" />
+    <limit lower="-1.0" upper="1.0" effort="10" velocity="1000" />
   </joint>
   <xacro:steering_hinge_transmission name="left_steering_hinge" />
@@ -100,5 +100,5 @@
     <child link="right_steering_hinge" />
     <axis xyz="-1 0 0" />
-    <limit lower="-1.0" upper="1.0" effort="10" velocity="100" />
+    <limit lower="-1.0" upper="1.0" effort="10" velocity="1000" />
   </joint>
   <xacro:steering_hinge_transmission name="right_steering_hinge" />
@@ -121,5 +121,5 @@
     <child link="left_front_wheel" />
     <axis xyz="0 0 -1" />
-    <limit effort="10" velocity="100" />
+    <limit effort="10" velocity="1000" />
   </joint>
   <xacro:wheel_transmission name="left_front_wheel" />
@@ -142,5 +142,5 @@
     <child link="right_front_wheel" />
     <axis xyz="0 0 -1" />
-    <limit effort="10" velocity="100"/>
+    <limit effort="10" velocity="1000"/>
   </joint>
   <xacro:wheel_transmission name="right_front_wheel" />

Commit message: Controllers issue solved

File: src/racecar-simulator/racecar_description/urdf/racecar_2.xacro (robot description, xacro)
@@ -43,5 +43,5 @@
     <child link="left_rear_wheel" />
     <axis xyz="0 0 -1" />
-    <limit effort="10" velocity="1000" />
+    <limit effort="10" velocity="100" />
   </joint>
   <xacro:wheel_transmission name="left_rear_wheel" />
@@ -64,5 +64,5 @@
     <child link="right_rear_wheel" />
     <axis xyz="0 0 -1" />
-    <limit effort="10" velocity="1000" />
+    <limit effort="10" velocity="100" />
   </joint>
   <xacro:wheel_transmission name="right_rear_wheel" />
@@ -82,5 +82,5 @@
     <child link="left_steering_hinge" />
     <axis xyz="-1 0 0" />
-    <limit lower="-1.0" upper="1.0" effort="10" velocity="1000" />
+    <limit lower="-1.0" upper="1.0" effort="10" velocity="100" />
   </joint>
   <xacro:steering_hinge_transmission name="left_steering_hinge" />
@@ -100,5 +100,5 @@
     <child link="right_steering_hinge" />
     <axis xyz="-1 0 0" />
-    <limit lower="-1.0" upper="1.0" effort="10" velocity="1000" />
+    <limit lower="-1.0" upper="1.0" effort="10" velocity="100" />
   </joint>
   <xacro:steering_hinge_transmission name="right_steering_hinge" />
@@ -121,5 +121,5 @@
     <child link="left_front_wheel" />
     <axis xyz="0 0 -1" />
-    <limit effort="10" velocity="1000" />
+    <limit effort="10" velocity="100" />
   </joint>
   <xacro:wheel_transmission name="left_front_wheel" />
@@ -142,5 +142,5 @@
     <child link="right_front_wheel" />
     <axis xyz="0 0 -1" />
-    <limit effort="10" velocity="1000"/>
+    <limit effort="10" velocity="100"/>
   </joint>
   <xacro:wheel_transmission name="right_front_wheel" />
